File: IVSense.sch (EAGLE design)
At the start: 14 parts

Commit message: update with schematic image
Parts:
- removed R3, R4: 1k, resistor:R-US_0204/5
- removed U$3: ARDUINO-BPLACE, adafruit:ARDUINO-BPLACE
- added C1, C2, C3: 0.1uF, adafruit:C-US025-025X050
- added R1_SHOULDER: 1k, resistor:R-US_0204/5
- added R2_SHOULDER, RF_SHOULDER, RF_SHOULDER1: 10k, resistor:R-US_0204/5
- R2_ELBOW: value 1k -> 10k
- RSENSE_ELBOW, RSENSE_SHOULDER: value 0.1 -> 0.1R
- renumbered R1 to R1_ELBOW, R2 to R2_ELBOW
Connections:
- new net N$10: RF_SHOULDER1.1
- new net N$11: C3.2
- new net N$12: C2.2
- new net N$13: R2_ELBOW.2
- new net N$14: MAX9918_ELBOW.OUT
- new net N$15: R2_SHOULDER.2
- new net N$16: MAX9918_SHOULDER.OUT
- new net N$3: U$1.5V
- new net N$4: R5.1
- new net N$6: U$1.GND
- new net N$7: C1.2
- new net N$9: RF_SHOULDER.1
- net A0: no longer U$3.A0
- net A1: no longer MAX9918_ELBOW.OUT, R2_ELBOW.2, U$3.A1
- net A2: now also C3.1, RF_SHOULDER1.2; no longer MAX9918_SHOULDER.OUT, R3.2, U$3.A2
- net A3: now also C2.1, RF_SHOULDER.2; no longer MAX9918_ELBOW.RS+, RSENSE_ELBOW.2, U$3.A3, U$4.OUT
- net A4: now also MAX9918_ELBOW.RS+, RSENSE_ELBOW.2, U$4.OUT; no longer MAX9918_SHOULDER.RS+, RSENSE_SHOULDER.2, U$3.A4, U$5.OUT
- net A5: now also MAX9918_SHOULDER.RS+, RSENSE_SHOULDER.2, U$5.OUT; no longer U$3.A5
- net GND: no longer U$3.GND
- net N$2: now also R1_SHOULDER.2, R2_SHOULDER.1; no longer R3.1, R4.2
- net N$5: now also R1_SHOULDER.1; no longer R4.1
- net VCC: now also C1.1; no longer R5.1, U$3.5V
Other:
- moved on the sheet: R5, R6, RSENSE_SHOULDER

Commit message: update
Parts:
- removed U$1: MOTOR_SHIELD, CAP:MOTOR_SHIELD
Connections:
- removed net A0: U$1.A0
- removed net A1: U$1.A1
- removed net A4: MAX9918_ELBOW.RS+, RSENSE_ELBOW.2, U$1.A4, U$4.OUT
- removed net A5: MAX9918_SHOULDER.RS+, RSENSE_SHOULDER.2, U$1.A5, U$5.OUT
- net A2: no longer U$1.A2
- net A3: no longer U$1.A3
- net GND: no longer MAX9918_ELBOW.SHDN, MAX9918_SHOULDER.SHDN
- net N$3: now also MAX9918_ELBOW.RS+, RSENSE_ELBOW.2, U$4.OUT; no longer U$1.5V
- net N$6: now also MAX9918_SHOULDER.RS+, RSENSE_SHOULDER.2, U$5.OUT; no longer U$1.GND
Other:
- note removed: "MOTOR POWER +"
- note removed: "MOTOR POWER -"
- moved on the sheet: C1, C2, C3, R1_ELBOW, R1_SHOULDER, R2_ELBOW, R2_SHOULDER, R5, R6, RF_SHOULDER, RF_SHOULDER1, RSENSE_ELBOW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

Commit message: update
Parts:
- RF_E, RF_S: value 10k -> 4.7k
- renumbered R1_ELBOW to RA_E, R1_SHOULDER to RA_S, R2_ELBOW to RB_E, R2_SHOULDER to RB_S, RF_SHOULDER to RF_S, RF_SHOULDER1 to RF_E, RSENSE_ELBOW to RSENSE_E, RSENSE_SHOULDER to RSENSE_S
Connections:
- removed net N$11: C3.2
- removed net N$12: C2.2
- removed net N$4: R5.1
- removed net N$7: C1.2
- net 2.5V: no longer MAX9918_ELBOW.GND, MAX9918_SHOULDER.GND
- net GND: now also C1.2, C2.2, C3.2, MAX9918_ELBOW.GND, MAX9918_SHOULDER.GND
- net VCC: now also R5.1
Other:
- note added: "FB"
- note added: "OUT"
- note added: "REFIN"
- note added: "RS+"
- note added: "RS-"
- note added: "SHDN"
